Commit message: Updated patrol system with detection, red zone logic, and README

File: install/night_patrol_robot/share/night_patrol_robot/urdf/patrol_robot.urdf.xacro (robot description, xacro)
@@ -1,172 +1 @@
-<?xml version="1.0"?>
-<robot name="patrol_robot" xmlns:xacro="http://www.ros.org/wiki/xacro">
-  <material name="blue"><color rgba="0.1 0.3 0.8 1"/></material>
-  <material name="black"><color rgba="0.05 0.05 0.05 1"/></material>
-  <material name="red"><color rgba="0.8 0.1 0.1 1"/></material>
-  <material name="dark_grey"><color rgba="0.2 0.2 0.2 1"/></material>
-  <link name="base_footprint"/>
-  <joint name="base_footprint_joint" type="fixed">
-    <parent link="base_footprint"/>
-    <child link="base_link"/>
-    <origin xyz="0 0 0.08" rpy="0 0 0"/>
-  </joint>
-  <link name="base_link">
-    <visual>
-      <geometry><box size="0.4 0.3 0.15"/></geometry>
-      <material name="blue"/>
-    </visual>
-    <collision>
-      <geometry><box size="0.4 0.3 0.15"/></geometry>
-    </collision>
-    <inertial>
-      <mass value="5.0"/>
-      <inertia ixx="0.05" ixy="0" ixz="0" iyy="0.05" iyz="0" izz="0.08"/>
-    </inertial>
-  </link>
-  <!-- Left wheel -->
-  <link name="left_wheel">
-    <visual>
-      <geometry><cylinder radius="0.08" length="0.04"/></geometry>
-      <material name="black"/>
-    </visual>
-    <collision>
-      <geometry><cylinder radius="0.08" length="0.04"/></geometry>
-    </collision>
-    <inertial>
-      <mass value="0.5"/>
-      <inertia ixx="0.001" ixy="0" ixz="0" iyy="0.001" iyz="0" izz="0.002"/>
-    </inertial>
-  </link>
-  <joint name="left_wheel_joint" type="continuous">
-    <parent link="base_link"/>
-    <child link="left_wheel"/>
-    <origin xyz="0 0.175 -0.02" rpy="-1.5708 0 0"/>
-    <axis xyz="0 0 1"/>
-  </joint>
-  <!-- Right wheel -->
-  <link name="right_wheel">
-    <visual>
-      <geometry><cylinder radius="0.08" length="0.04"/></geometry>
-      <material name="black"/>
-    </visual>
-    <collision>
-      <geometry><cylinder radius="0.08" length="0.04"/></geometry>
-    </collision>
-    <inertial>
-      <mass value="0.5"/>
-      <inertia ixx="0.001" ixy="0" ixz="0" iyy="0.001" iyz="0" izz="0.002"/>
-    </inertial>
-  </link>
-  <joint name="right_wheel_joint" type="continuous">
-    <parent link="base_link"/>
-    <child link="right_wheel"/>
-    <origin xyz="0 -0.175 -0.02" rpy="-1.5708 0 0"/>
-    <axis xyz="0 0 1"/>
-  </joint>
-  <!-- Caster -->
-  <link name="caster_wheel">
-    <visual><geometry><sphere radius="0.03"/></geometry><material name="dark_grey"/></visual>
-    <collision><geometry><sphere radius="0.03"/></geometry></collision>
-    <inertial>
-      <mass value="0.2"/>
-      <inertia ixx="0.0001" ixy="0" ixz="0" iyy="0.0001" iyz="0" izz="0.0001"/>
-    </inertial>
-  </link>
-  <joint name="caster_joint" type="fixed">
-    <parent link="base_link"/>
-    <child link="caster_wheel"/>
-    <origin xyz="-0.15 0 -0.06" rpy="0 0 0"/>
-  </joint>
-  <!-- LiDAR -->
-  <link name="lidar_link">
-    <visual><geometry><cylinder radius="0.04" length="0.05"/></geometry><material name="red"/></visual>
-    <collision><geometry><cylinder radius="0.04" length="0.05"/></geometry></collision>
-    <inertial>
-      <mass value="0.1"/>
-      <inertia ixx="0.0001" ixy="0" ixz="0" iyy="0.0001" iyz="0" izz="0.0001"/>
-    </inertial>
-  </link>
-  <joint name="lidar_joint" type="fixed">
-    <parent link="base_link"/>
-    <child link="lidar_link"/>
-    <origin xyz="0 0 0.1" rpy="0 0 0"/>
-  </joint>
-  <!-- Camera -->
-  <link name="camera_link">
-    <visual><geometry><box size="0.04 0.08 0.04"/></geometry><material name="dark_grey"/></visual>
-    <collision><geometry><box size="0.04 0.08 0.04"/></geometry></collision>
-    <inertial>
-      <mass value="0.05"/>
-      <inertia ixx="0.00001" ixy="0" ixz="0" iyy="0.00001" iyz="0" izz="0.00001"/>
-    </inertial>
-  </link>
-  <joint name="camera_joint" type="fixed">
-    <parent link="base_link"/>
-    <child link="camera_link"/>
-    <origin xyz="0.18 0 0.05" rpy="0 0 0"/>
-  </joint>
-  <!-- GAZEBO PLUGINS -->
-  <gazebo>
-    <plugin filename="gz-sim-diff-drive-system"
-            name="gz::sim::systems::DiffDrive">
-      <left_joint>left_wheel_joint</left_joint>
-      <right_joint>right_wheel_joint</right_joint>
-      <wheel_separation>0.35</wheel_separation>
-      <wheel_radius>0.08</wheel_radius>
-      <odom_publish_frequency>20</odom_publish_frequency>
-      <topic>/cmd_vel</topic>
-      <odom_topic>/odom</odom_topic>
-      <tf_topic>/tf</tf_topic>
-      <frame_id>odom</frame_id>
-      <child_frame_id>base_footprint</child_frame_id>
-      <min_acceleration>-1</min_acceleration>
-      <max_acceleration>1</max_acceleration>
-    </plugin>
-  </gazebo>
-  <gazebo>
-    <plugin filename="gz-sim-joint-state-publisher-system"
-            name="gz::sim::systems::JointStatePublisher"/>
-  </gazebo>
-  <!-- LiDAR sensor -->
-  <gazebo reference="lidar_link">
-    <sensor name="lidar" type="gpu_lidar">
-      <topic>/scan</topic>
-      <update_rate>10</update_rate>
-      <lidar>
-        <scan>
-          <horizontal>
-            <samples>360</samples>
-            <resolution>1</resolution>
-            <min_angle>-3.14159</min_angle>
-            <max_angle>3.14159</max_angle>
-          </horizontal>
-        </scan>
-        <range>
-          <min>0.12</min>
-          <max>10.0</max>
-          <resolution>0.01</resolution>
-        </range>
-      </lidar>
-      <always_on>true</always_on>
-      <visualize>true</visualize>
-    </sensor>
-  </gazebo>
-  <!-- Camera sensor -->
-  <gazebo reference="camera_link">
-    <sensor name="camera" type="camera">
-      <topic>/camera/image_raw</topic>
-      <update_rate>15</update_rate>
-      <camera>
-        <horizontal_fov>1.047</horizontal_fov>
-        <image>
-          <width>640</width>
-          <height>480</height>
-          <format>R8G8B8</format>
-        </image>
-        <clip><near>0.1</near><far>100</far></clip>
-      </camera>
-      <always_on>true</always_on>
-      <visualize>true</visualize>
-    </sensor>
-  </gazebo>
-</robot>
+/mnt/c/Users/LENOVO/OneDrive/Desktop/ros2_ws/src/night_patrol_robot/urdf/patrol_robot.urdf.xacro
